File: shitbox.kicad_sch (KiCad schematic)
At the start: 17 parts, among them U1 Raspberry_Pi_Pico

Commit message: Happy with the positioning of the buttons. Now to updating the wiring.
Parts:
- S13, S14, S15, S16: footprint PCM_Switch_Keyboard_Hotswap_Kailh:SW_Hotswap_Kailh_MX -> Button Switch:SW_PUSH_6mm
Changed lines of the file:
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@@
 			)
 		)
-		(property "Footprint" "PCM_Switch_Keyboard_Hotswap_Kailh:SW_Hotswap_Kailh_MX"
+		(property "Footprint" "Button Switch:SW_PUSH_6mm"
 			(at 127 128.27 0)
 			(effects
@@
 			)
 		)
-		(property "Footprint" "PCM_Switch_Keyboard_Hotswap_Kailh:SW_Hotswap_Kailh_MX"
+		(property "Footprint" "Button Switch:SW_PUSH_6mm"
 			(at 135.89 135.89 0)
 			(effects
@@
 			)
 		)
-		(property "Footprint" "PCM_Switch_Keyboard_Hotswap_Kailh:SW_Hotswap_Kailh_MX"
+		(property "Footprint" "Button Switch:SW_PUSH_6mm"
 			(at 119.38 120.65 0)
 			(effects
@@
 			)
 		)
-		(property "Footprint" "PCM_Switch_Keyboard_Hotswap_Kailh:SW_Hotswap_Kailh_MX"
+		(property "Footprint" "Button Switch:SW_PUSH_6mm"
 			(at 144.78 144.78 0)
 			(effects
