File: shitbox.kicad_pcb (KiCad board)
At the start: 2 copper layers, 17 parts, among them U1 Raspberry_Pi_Pico

Commit message: Happy with the positioning of the buttons. Now to updating the wiring.
Parts:
- added REF**: MountingHole_3.2mm_Pad, PCM_SL_Mechanical:MountingHole_3.2mm_Pad, F.Cu at (175.0, 105.0)
- added REF**: MountingHole_3.2mm_Pad, PCM_SL_Mechanical:MountingHole_3.2mm_Pad, F.Cu at (61.0, 110.0)
- added REF**: MountingHole_3.2mm_Pad, PCM_SL_Mechanical:MountingHole_3.2mm_Pad, F.Cu at (113.0, 74.0)
- added REF**: MountingHole_3.2mm_Pad, PCM_SL_Mechanical:MountingHole_3.2mm_Pad, F.Cu at (11.5, 25.5)
- added REF**: MountingHole_3.2mm_Pad, PCM_SL_Mechanical:MountingHole_3.2mm_Pad, F.Cu at (181.0, 26.0)
- S13, S14, S15, S16: footprint PCM_Switch_Keyboard_Hotswap_Kailh:SW_Hotswap_Kailh_MX -> Button Switch:SW_PUSH_6mm
- moved S13 371.7 mm to (67.2, 3.25)
- moved S14 361.9 mm to (77.0, 3.25)
- moved S15 350.4 mm to (86.5, 3.25)
- moved S16 339.6 mm to (96.2, 3.25)
- moved U1 337.4 mm to (188.1, 75.1)
- moved S7 335.1 mm to (151.5, 46.0)
- moved S12 335.1 mm to (169.5, 31.5)
- moved S6 335.1 mm to (128.5, 48.0)
- moved S1 334.9 mm to (64.1, 98.2)
- moved S8 334.6 mm to (98.4, 99.5)
- moved S3 334.5 mm to (65.3, 43.8)
- moved S5 334.5 mm to (109.9, 62.1)
- moved S10 334.4 mm to (120.0, 25.0)
- moved S11 334.4 mm to (143.0, 23.0)
- moved S9 334.2 mm to (101.0, 38.5)
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Routing:
- net Net-(U1-GPIO8): track 307.2 -> 0.00 mm
- net Net-(U1-GPIO13): track 304.1 -> 0.00 mm
- net Net-(U1-GPIO4): track 191.1 -> 0.00 mm
- net Net-(U1-GPIO5): track 178.1 -> 0.00 mm
- net Net-(U1-GPIO3): track 156.2 -> 0.00 mm
- net Net-(U1-GPIO2): track 137.0 -> 0.00 mm
- net Net-(U1-GPIO9): track 84.9 -> 0.00 mm
- net Net-(U1-GPIO7): track 83.9 -> 0.00 mm
- net Net-(U1-GPIO6): track 68.7 -> 0.00 mm
- net Net-(S1-Pad2): track 1.41 -> 0.00 mm
Other:
- board outline added: 190 x 120 mm

Commit message: Kicad, please don't crash...
Parts:
- moved S13 35.8 mm to (102.8, 7.75), turned to 180 degrees
- moved S16 22.9 mm to (73.8, 7.75), turned to 180 degrees
- moved S14 16.6 mm to (93.0, 7.75), turned to 180 degrees
- moved S15 5.41 mm to (83.5, 7.75), turned to 180 degrees
Routing:
- net Net-(S1-Pad2): track 0.00 -> 587.2 mm, vias 0 -> 3
- net Net-(U1-GPIO4): track 0.00 -> 258.7 mm
- net Net-(U1-GPIO5): track 0.00 -> 250.6 mm
- net Net-(U1-GPIO3): track 0.00 -> 216.8 mm
- net Net-(U1-GPIO21): track 0.00 -> 161.1 mm
- net Net-(U1-GPIO20): track 0.00 -> 146.7 mm
- net Net-(U1-GPIO17): track 0.00 -> 144.1 mm
- net Net-(U1-GPIO2): track 0.00 -> 130.4 mm
- net Net-(U1-GPIO16): track 0.00 -> 129.9 mm
- net Net-(U1-GPIO7): track 0.00 -> 103.1 mm
- net Net-(U1-GPIO9): track 0.00 -> 95.6 mm, vias 0 -> 1
- net Net-(U1-GPIO10): track 0.00 -> 83.2 mm, vias 0 -> 1
- net Net-(U1-GPIO11): track 0.00 -> 72.9 mm, vias 0 -> 1
- net Net-(U1-GPIO6): track 0.00 -> 71.7 mm
- net Net-(U1-GPIO13): track 0.00 -> 60.7 mm, vias 0 -> 1
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- added copper zone on B.Cu, net (none)
- added copper zone on F.Cu, net (none)
Other:
- outline, holes or cut-outs redrawn
- board text added: "Blamed the beast - jiji"
